File: PS-33D-Adapter.kicad_pcb (KiCad board)
At the start: 2 copper layers, 8 parts, among them J1 CONN_05, J2 Conn_02x04_Counter_Clockwise, Q1 MOSFET-NCH-BSS138, Q2 MOSFET-NCH-BSS138

Commit message: feat: update mask clearance, mask min width
Other:
- rule pad_to_mask_clearance: 0 -> 0.0508

Commit message: feat: update setup
Other:
- net class Default: clearance 0.2 -> 0.254; trace_width 0.25 -> 0.254; via_dia 0.8 -> 0.762; via_drill 0.4 -> 0.381
- rule trace_clearance: 0.2 -> 0.254
- rule trace_min: 0.2 -> 0.1524
- rule via_min_drill: 0.3 -> 0.254
- rule via_min_size: 0.4 -> 0.508

Commit message: feat: update pcb
Parts:
- moved R3 14.6 mm to (151.6, 77.5)
- moved Q2 12.8 mm to (155.9, 78.7), turned to 270 degrees
- moved R4 12.5 mm to (151.6, 82.5)
- moved R2 12.3 mm to (151.6, 85.1)
- moved R1 12.0 mm to (151.6, 80.0)
- moved Q1 11.9 mm to (155.9, 83.8), turned to 270 degrees
- moved J1 8.32 mm to (147.3, 78.7)
- moved J2 5.32 mm to (160.0, 78.7)

Commit message: feat: update pcb
Parts:
- moved R2 2.54 mm to (151.6, 82.5)
- moved Q1 1.59 mm to (155.9, 82.2)
- moved R3 1.27 mm to (151.6, 78.7)
- moved R4 1.27 mm to (151.6, 81.3)
Other:
- board outline added: 19.1 x 10.2 mm

Commit message: feat: update pcb
Parts:
- moved J2 2.54 mm to (157.5, 78.7)
- moved Q1 2.01 mm to (154.0, 82.9)
- moved Q2 1.93 mm to (154.0, 79.1)
- moved R2 1.32 mm to (150.7, 83.6)
- moved R4 1.14 mm to (150.7, 82.0)
- moved R3 0.88 mm to (150.7, 78.5)
- moved R1 0.84 mm to (150.7, 80.0)
Other:
- board outline removed
- net class Default: clearance 0.254 -> 0.15; trace_width 0.254 -> 0.25; via_dia 0.762 -> 0.6; via_drill 0.381 -> 0.3
- rule trace_clearance: 0.254 -> 0.15
- rule trace_min: 0.1524 -> 0.16
- rule via_min_drill: 0.254 -> 0.3
- rule via_min_size: 0.508 -> 0.6
Changed lines of the file:
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@@
   (general
     (thickness 1.6)
-    (drawings 4)
+    (drawings 0)
     (tracks 0)
     (zones 0)
@@
   )
   (setup
-    (last_trace_width 0.254)
-    (trace_clearance 0.254)
+    (last_trace_width 0.25)
+    (trace_clearance 0.15)
     (zone_clearance 0.508)
     (zone_45_only no)
-    (trace_min 0.1524)
-    (via_size 0.762)
-    (via_drill 0.381)
-    (via_min_size 0.508)
-    (via_min_drill 0.254)
+    (trace_min 0.16)
+    (via_size 0.6)
+    (via_drill 0.3)
+    (via_min_size 0.6)
+    (via_min_drill 0.3)
     (uvia_size 0.762)
     (uvia_drill 0.381)
@@
   (net 7 SCL)
   (net_class Default "This is the default net class."
-    (clearance 0.254)
-    (trace_width 0.254)
-    (via_dia 0.762)
-    (via_drill 0.381)
+    (clearance 0.15)
+    (trace_width 0.25)
+    (via_dia 0.6)
+    (via_drill 0.3)
     (uvia_dia 0.762)
     (uvia_drill 0.381)
@@
   )
   (module Connector_PinHeader_1.27mm:PinHeader_2x04_P1.27mm_Vertical (layer F.Cu)
-    (at 160.02 78.74)
+    (at 157.48 78.74)
     (descr "Through hole straight pin header, 2x04, 1.27mm pitch, double rows")
     (tags "Through hole pin header THT 2x04 1.27mm double row")
@@
   )
   (module Silicon-Standard:SOT23-3 (layer F.Cu)
-    (at 155.93822 82.22996 270)
+    (at 154.03322 82.87004 270)
     (descr SOT23-3)
     (tags SOT23-3)
@@
   )
   (module Silicon-Standard:SOT23-3 (layer F.Cu)
-    (at 155.93822 78.74 270)
+    (at 154.03322 79.06004 270)
     (descr SOT23-3)
     (tags SOT23-3)
@@
   )
   (module Resistors:0603 (layer F.Cu)
-    (at 151.55164 80.01)
+    (at 150.70836 80.01)
     (descr "GENERIC 1608 (0603) PACKAGE")
     (tags "GENERIC 1608 (0603) PACKAGE")
@@
   )
   (module Resistors:0603 (layer F.Cu)
-    (at 151.55164 82.55)
+    (at 150.70836 83.566)
     (descr "GENERIC 1608 (0603) PACKAGE")
     (tags "GENERIC 1608 (0603) PACKAGE")
@@
   )
   (module Resistors:0603 (layer F.Cu)
-    (at 151.55164 78.74)
+    (at 150.70836 78.486)
     (descr "GENERIC 1608 (0603) PACKAGE")
     (tags "GENERIC 1608 (0603) PACKAGE")
@@
   )
   (module Resistors:0603 (layer F.Cu)
-    (at 151.55164 81.28)
+    (at 150.70836 82.042)
     (descr "GENERIC 1608 (0603) PACKAGE")
     (tags "GENERIC 1608 (0603) PACKAGE")
@@
       (net 2 5V) (solder_mask_margin 0.1016))
   )
-  (gr_line (start 144.78 86.36) (end 144.78 76.2) (layer Edge.Cuts) (width 0.05))
-  (gr_line (start 163.83 86.36) (end 144.78 86.36) (layer Edge.Cuts) (width 0.05))
-  (gr_line (start 163.83 76.2) (end 163.83 86.36) (layer Edge.Cuts) (width 0.05))
-  (gr_line (start 144.78 76.2) (end 163.83 76.2) (layer Edge.Cuts) (width 0.05))
 )

Commit message: feat: arrange parts
Parts:
- moved J2 0.76 mm to (157.5, 79.5)
- moved Q2 0.76 mm to (154.0, 79.8)
- moved R1 0.51 mm to (150.7, 80.5)
- moved R3 0.51 mm to (150.7, 79.0)
Other:
- board outline added: 15 x 7.6 mm

Commit message: feat: update pcb
Routing:
- net 5V: track 0.00 -> 5.65 mm
- net 3V3: track 0.00 -> 4.65 mm, vias 0 -> 1
Changed lines of the file:
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@@
     (thickness 1.6)
     (drawings 4)
-    (tracks 0)
+    (tracks 13)
     (zones 0)
     (modules 8)
@@
   )
   (setup
-    (last_trace_width 0.25)
+    (last_trace_width 0.3)
+    (user_trace_width 0.3)
     (trace_clearance 0.15)
     (zone_clearance 0.508)
@@
   (gr_line (start 160.528 77.47) (end 160.528 85.09) (layer Edge.Cuts) (width 0.05))
   (gr_line (start 145.542 77.47) (end 160.528 77.47) (layer Edge.Cuts) (width 0.05))
+  (segment (start 147.32 80.01) (end 147.574 80.01) (width 0.3) (layer F.Cu) (net 2))
+  (segment (start 147.574 80.01) (end 148.120001 80.556001) (width 0.3) (layer F.Cu) (net 2))
+  (segment (start 148.120001 80.556001) (end 148.120001 81.826001) (width 0.3) (layer F.Cu) (net 2))
+  (segment (start 148.336 82.042) (end 149.86 82.042) (width 0.3) (layer F.Cu) (net 2))
+  (segment (start 148.120001 81.826001) (end 148.336 82.042) (width 0.3) (layer F.Cu) (net 2))
+  (segment (start 149.86 82.042) (end 149.86 83.566) (width 0.3) (layer F.Cu) (net 2))
+  (via (at 148.629651 80.239366) (size 0.6) (drill 0.3) (layers F.Cu B.Cu) (net 3))
+  (segment (start 147.589017 81.28) (end 148.629651 80.239366) (width 0.3) (layer B.Cu) (net 3))
+  (segment (start 147.32 81.28) (end 147.589017 81.28) (width 0.3) (layer B.Cu) (net 3))
+  (segment (start 148.629651 80.239366) (end 148.629651 80.303651) (width 0.3) (layer F.Cu) (net 3))
+  (segment (start 148.844 80.518) (end 149.86 80.518) (width 0.3) (layer F.Cu) (net 3))
+  (segment (start 148.629651 80.303651) (end 148.844 80.518) (width 0.3) (layer F.Cu) (net 3))
+  (segment (start 149.86 80.518) (end 149.86 78.994) (width 0.3) (layer F.Cu) (net 3))
 )

Commit message: feat: update schematic, pcb
Parts:
- turned Q1 to 90 degrees
- turned Q2 to 90 degrees
Connections:
- J2 pad 2: SDA -> 3V3
- J2 pad 3: SCL -> SDA
- J2 pad 4: GND -> SDA
- J2 pad 5: GND -> SCL
- J2 pad 7: SDA -> GND
- J2 pad 8: 3V3 -> GND
Routing:
- net SDA: track 0.00 -> 1.27 mm
- net SCL: track 0.00 -> 1.27 mm
- net 3V3: track 4.65 -> 5.92 mm
Changed lines of the file:
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@@
     (thickness 1.6)
     (drawings 4)
-    (tracks 13)
+    (tracks 16)
     (zones 0)
     (modules 8)
@@
       (net 3 3V3))
     (pad 2 thru_hole oval (at 1.27 0) (size 1 1) (drill 0.65) (layers *.Cu *.Mask)
+      (net 3 3V3))
+    (pad 3 thru_hole oval (at 0 1.27) (size 1 1) (drill 0.65) (layers *.Cu *.Mask)
       (net 6 SDA))
-    (pad 3 thru_hole oval (at 0 1.27) (size 1 1) (drill 0.65) (layers *.Cu *.Mask)
+    (pad 4 thru_hole oval (at 1.27 1.27) (size 1 1) (drill 0.65) (layers *.Cu *.Mask)
+      (net 6 SDA))
+    (pad 5 thru_hole oval (at 0 2.54) (size 1 1) (drill 0.65) (layers *.Cu *.Mask)
       (net 7 SCL))
-    (pad 4 thru_hole oval (at 1.27 1.27) (size 1 1) (drill 0.65) (layers *.Cu *.Mask)
-      (net 1 GND))
-    (pad 5 thru_hole oval (at 0 2.54) (size 1 1) (drill 0.65) (layers *.Cu *.Mask)
-      (net 1 GND))
     (pad 6 thru_hole oval (at 1.27 2.54) (size 1 1) (drill 0.65) (layers *.Cu *.Mask)
       (net 7 SCL))
     (pad 7 thru_hole oval (at 0 3.81) (size 1 1) (drill 0.65) (layers *.Cu *.Mask)
-      (net 6 SDA))
+      (net 1 GND))
     (pad 8 thru_hole oval (at 1.27 3.81) (size 1 1) (drill 0.65) (layers *.Cu *.Mask)
-      (net 3 3V3))
+      (net 1 GND))
     (model ${KISYS3DMOD}/Connector_PinHeader_1.27mm.3dshapes/PinHeader_2x04_P1.27mm_Vertical.wrl
       (at (xyz 0 0 0))
@@
   )
   (module Silicon-Standard:SOT23-3 (layer F.Cu)
-    (at 154.03322 82.87004 270)
+    (at 154.03322 82.87004 90)
     (descr SOT23-3)
     (tags SOT23-3)
@@
     (fp_line (start 0.79756 -0.6985) (end 1.39954 -0.6985) (layer F.SilkS) (width 0.2032))
     (fp_line (start 1.39954 -0.6985) (end 1.39954 0.09906) (layer F.SilkS) (width 0.2032))
-    (pad 1 smd rect (at -0.94996 0.99822 270) (size 0.79756 0.89916) (layers F.Cu F.Paste F.Mask)
+    (pad 1 smd rect (at -0.94996 0.99822 90) (size 0.79756 0.89916) (layers F.Cu F.Paste F.Mask)
       (net 3 3V3) (solder_mask_margin 0.1016))
-    (pad 2 smd rect (at 0.94996 0.99822 270) (size 0.79756 0.89916) (layers F.Cu F.Paste F.Mask)
+    (pad 2 smd rect (at 0.94996 0.99822 90) (size 0.79756 0.89916) (layers F.Cu F.Paste F.Mask)
       (net 6 SDA) (solder_mask_margin 0.1016))
-    (pad 3 smd rect (at 0 -1.09982 270) (size 0.79756 0.89916) (layers F.Cu F.Paste F.Mask)
+    (pad 3 smd rect (at 0 -1.09982 90) (size 0.79756 0.89916) (layers F.Cu F.Paste F.Mask)
       (net 5 M.SDA) (solder_mask_margin 0.1016))
   )
   (module Silicon-Standard:SOT23-3 (layer F.Cu)
-    (at 154.03322 79.82204 270)
+    (at 154.03322 79.82204 90)
     (descr SOT23-3)
     (tags SOT23-3)
@@
     (fp_line (start 1.4224 0.6604) (end -1.4224 0.6604) (layer Dwgs.User) (width 0.1524))
     (fp_line (start 1.4224 -0.6604) (end 1.4224 0.6604) (layer Dwgs.User) (width 0.1524))
-    (pad 3 smd rect (at 0 -1.09982 270) (size 0.79756 0.89916) (layers F.Cu F.Paste F.Mask)
+    (pad 3 smd rect (at 0 -1.09982 90) (size 0.79756 0.89916) (layers F.Cu F.Paste F.Mask)
       (net 4 M.SCL) (solder_mask_margin 0.1016))
-    (pad 2 smd rect (at 0.94996 0.99822 270) (size 0.79756 0.89916) (layers F.Cu F.Paste F.Mask)
+    (pad 2 smd rect (at 0.94996 0.99822 90) (size 0.79756 0.89916) (layers F.Cu F.Paste F.Mask)
       (net 7 SCL) (solder_mask_margin 0.1016))
-    (pad 1 smd rect (at -0.94996 0.99822 270) (size 0.79756 0.89916) (layers F.Cu F.Paste F.Mask)
+    (pad 1 smd rect (at -0.94996 0.99822 90) (size 0.79756 0.89916) (layers F.Cu F.Paste F.Mask)
       (net 3 3V3) (solder_mask_margin 0.1016))
   )
@@
   (segment (start 148.629651 80.303651) (end 148.844 80.518) (width 0.3) (layer F.Cu) (net 3))
   (segment (start 149.86 80.518) (end 149.86 78.994) (width 0.3) (layer F.Cu) (net 3))
+  (segment (start 157.48 79.502) (end 158.75 79.502) (width 0.3) (layer F.Cu) (net 3))
+  (segment (start 157.48 80.772) (end 158.75 80.772) (width 0.25) (layer F.Cu) (net 6))
+  (segment (start 157.48 82.042) (end 158.75 82.042) (width 0.25) (layer F.Cu) (net 7))
 )
