File: PS-33D-Adapter.kicad_pcb (KiCad board)
At the start: 2 copper layers, 15 x 7.6 mm, 8 parts, among them J1 CONN_05, J2 Conn_02x04_Counter_Clockwise, Q1 MOSFET-NCH-BSS138, Q2 MOSFET-NCH-BSS138

Commit message: feat: update pcb
Routing:
- net SCL: track 1.27 -> 14.4 mm, vias 0 -> 1
- net M.SCL: track 0.00 -> 10.6 mm, vias 0 -> 3
- net M.SDA: track 0.00 -> 8.42 mm, vias 0 -> 2
- net SDA: track 1.27 -> 9.40 mm, vias 0 -> 1
- net 3V3: track 5.92 -> 12.7 mm
Other:
- net class Default: trace_width 0.25 -> 0.2

Commit message: feat: add copper pour
Routing:
- net 3V3: track 12.7 -> 21.2 mm
- added copper zone on B.Cu, net GND
- added copper zone on F.Cu, net GND

Commit message: feat: update pcb
Other:
- board text added: "V 1.0"
