File: PS-33D-Adapter.sch (KiCad schematic (older format))
At the start: 8 parts, among them J1 CONN_05, J2 Conn_02x04_Counter_Clockwise, Q1 MOSFET-NCH-BSS138, Q2 MOSFET-NCH-BSS138

Commit message: feat: update schematic, pcb
Connections:
- net 3V3: now also J2.2 (Pin_2); no longer J2.8 (Pin_8)
- net GND: now also J2.7 (Pin_7), J2.8 (Pin_8); no longer J2.4 (Pin_4), J2.5 (Pin_5)
- net SCL: now also J2.5 (Pin_5); no longer J2.3 (Pin_3)
- net SDA: now also J2.3 (Pin_3), J2.4 (Pin_4); no longer J2.2 (Pin_2), J2.7 (Pin_7)
Changed lines of the file:
@@
 Comment4 ""
 $EndDescr
-$Comp
-L Connector_Generic:Conn_02x04_Counter_Clockwise J2
-U 1 1 618C7D19
-P 4250 3550
-F 0 "J2" H 4300 3867 50  0000 C CNN
-F 1 "Conn_02x04_Counter_Clockwise" H 4300 3776 50  0000 C CNN
-F 2 "Connector_PinHeader_1.27mm:PinHeader_2x04_P1.27mm_Vertical" H 4250 3550 50  0001 C CNN
-F 3 "~" H 4250 3550 50  0001 C CNN
-	1    4250 3550
-	1    0    0    -1
-$EndComp
-Wire Wire Line
-	4550 3450 4800 3450
-Wire Wire Line
-	4550 3550 4800 3550
-Wire Wire Line
-	4550 3650 4800 3650
-Wire Wire Line
-	4550 3750 4800 3750
-Wire Wire Line
-	4050 3450 3750 3450
-Wire Wire Line
-	4050 3550 3750 3550
-Wire Wire Line
-	4050 3650 3750 3650
-Wire Wire Line
-	4050 3750 3750 3750
-Text GLabel 3750 3550 0    50   Input ~ 0
-SDA
-Text GLabel 3750 3650 0    50   Input ~ 0
-SCL
-Text GLabel 3750 3750 0    50   Input ~ 0
-GND
-Text GLabel 4800 3550 2    50   Input ~ 0
-SDA
-Text GLabel 4800 3650 2    50   Input ~ 0
-SCL
-Text GLabel 4800 3750 2    50   Input ~ 0
-GND
+Wire Wire Line
+	4050 3450 3900 3450
+Wire Wire Line
+	4050 3650 3900 3650
 $Comp
 L SparkFun-DiscreteSemi:MOSFET-NCH-BSS138 Q1
@@
 Wire Wire Line
 	6350 3700 6200 3700
-Text GLabel 4800 3450 2    50   Input ~ 0
-3V3
 Text GLabel 3750 3450 0    50   Input ~ 0
 3V3
@@
 Wire Wire Line
 	8300 3000 8300 3050
+Wire Wire Line
+	4050 3550 3900 3550
+Wire Wire Line
+	3900 3550 3900 3450
+Connection ~ 3900 3450
+Wire Wire Line
+	3900 3450 3750 3450
+$Comp
+L Connector_Generic:Conn_02x04_Counter_Clockwise J2
+U 1 1 618C7D19
+P 4250 3550
+F 0 "J2" H 4300 3867 50  0000 C CNN
+F 1 "Conn_02x04_Counter_Clockwise" H 4300 3776 50  0000 C CNN
+F 2 "Connector_PinHeader_1.27mm:PinHeader_2x04_P1.27mm_Vertical" H 4250 3550 50  0001 C CNN
+F 3 "~" H 4250 3550 50  0001 C CNN
+	1    4250 3550
+	1    0    0    -1
+$EndComp
+Text GLabel 3750 3650 0    50   Input ~ 0
+SDA
+Wire Wire Line
+	4050 3750 3900 3750
+Wire Wire Line
+	3900 3750 3900 3650
+Connection ~ 3900 3650
+Wire Wire Line
+	3900 3650 3750 3650
+Text GLabel 4850 3750 2    50   Input ~ 0
+SCL
+Text GLabel 4850 3550 2    50   Input ~ 0
+GND
+Wire Wire Line
+	4550 3750 4700 3750
+Wire Wire Line
+	4550 3650 4700 3650
+Wire Wire Line
+	4700 3650 4700 3750
+Connection ~ 4700 3750
+Wire Wire Line
+	4550 3550 4700 3550
+Wire Wire Line
+	4550 3450 4700 3450
+Wire Wire Line
+	4700 3450 4700 3550
+Connection ~ 4700 3550
+Wire Wire Line
+	4700 3550 4850 3550
+Wire Wire Line
+	4700 3750 4850 3750
 $EndSCHEMATC

Commit message: feat: update footprints of connectors
Parts:
- J1: footprint Connector_PinHeader_1.27mm:PinHeader_1x05_P1.27mm_Vertical -> Connector_PinHeader_2.54mm:PinHeader_1x05_P2.54mm_Vertical
- J2: footprint Connector_PinHeader_1.27mm:PinHeader_2x04_P1.27mm_Vertical -> Connector_PinSocket_2.54mm:PinSocket_2x04_P2.54mm_Vertical
Changed lines of the file:
@@
 F 0 "J1" H 3708 3160 45  0000 C CNN
 F 1 "CONN_05" H 3708 3076 45  0000 C CNN
-F 2 "Connector_PinHeader_1.27mm:PinHeader_1x05_P1.27mm_Vertical" H 3750 3050 20  0001 C CNN
+F 2 "Connector_PinHeader_2.54mm:PinHeader_1x05_P2.54mm_Vertical" H 3750 3050 20  0001 C CNN
 F 3 "" H 3750 2450 50  0001 C CNN
 F 4 "XXX-00000" H 3708 2981 60  0000 C CNN "Field4"
@@
 F 0 "J2" H 4300 3867 50  0000 C CNN
 F 1 "Conn_02x04_Counter_Clockwise" H 4300 3776 50  0000 C CNN
-F 2 "Connector_PinHeader_1.27mm:PinHeader_2x04_P1.27mm_Vertical" H 4250 3550 50  0001 C CNN
+F 2 "Connector_PinSocket_2.54mm:PinSocket_2x04_P2.54mm_Vertical" H 4250 3550 50  0001 C CNN
 F 3 "~" H 4250 3550 50  0001 C CNN
 	1    4250 3550

Commit message: feat: update schematic, pcb
Parts:
- removed J2: Conn_02x04_Counter_Clockwise, Connector_PinSocket_2.54mm:PinSocket_2x04_P2.54mm_Vertical, symbol Connector_Generic:Conn_02x04_Counter_Clockwise
- added J1, J3: CONN_04, Connector_PinHeader_2.54mm:PinHeader_1x04_P2.54mm_Vertical, symbol SparkFun-Connectors:CONN_04
- renumbered J1 to J2
Connections:
- net 3V3: now also J1.4, J3.4
- net GND: now also J1.1, J3.1
- net SCL: now also J1.2, J3.2
- net SDA: now also J1.3, J3.3
Changed lines of the file:
@@
 Comment4 ""
 $EndDescr
-Wire Wire Line
-	4050 3450 3900 3450
-Wire Wire Line
-	4050 3650 3900 3650
 $Comp
 L SparkFun-DiscreteSemi:MOSFET-NCH-BSS138 Q1
@@
 $EndComp
 $Comp
-L SparkFun-Connectors:CONN_05 J1
+L SparkFun-Connectors:CONN_05 J2
 U 1 1 61A8E613
 P 3750 2450
-F 0 "J1" H 3708 3160 45  0000 C CNN
+F 0 "J2" H 3708 3160 45  0000 C CNN
 F 1 "CONN_05" H 3708 3076 45  0000 C CNN
 F 2 "Connector_PinHeader_2.54mm:PinHeader_1x05_P2.54mm_Vertical" H 3750 3050 20  0001 C CNN
@@
 Wire Wire Line
 	6350 3700 6200 3700
-Text GLabel 3750 3450 0    50   Input ~ 0
-3V3
 Text GLabel 6200 2850 1    50   Input ~ 0
 3V3
@@
 Wire Wire Line
 	8300 3000 8300 3050
-Wire Wire Line
-	4050 3550 3900 3550
-Wire Wire Line
-	3900 3550 3900 3450
-Connection ~ 3900 3450
-Wire Wire Line
-	3900 3450 3750 3450
-$Comp
-L Connector_Generic:Conn_02x04_Counter_Clockwise J2
-U 1 1 618C7D19
-P 4250 3550
-F 0 "J2" H 4300 3867 50  0000 C CNN
-F 1 "Conn_02x04_Counter_Clockwise" H 4300 3776 50  0000 C CNN
-F 2 "Connector_PinSocket_2.54mm:PinSocket_2x04_P2.54mm_Vertical" H 4250 3550 50  0001 C CNN
-F 3 "~" H 4250 3550 50  0001 C CNN
-	1    4250 3550
+$Comp
+L SparkFun-Connectors:CONN_04 J1
+U 1 1 61EE1982
+P 3650 3550
+F 0 "J1" H 3608 4160 45  0000 C CNN
+F 1 "CONN_04" H 3608 4076 45  0000 C CNN
+F 2 "Connector_PinHeader_2.54mm:PinHeader_1x04_P2.54mm_Vertical" H 3650 4050 20  0001 C CNN
+F 3 "" H 3650 3550 50  0001 C CNN
+F 4 "CONN-09696" H 3608 3981 60  0000 C CNN "Field4"
+	1    3650 3550
 	1    0    0    -1
 $EndComp
-Text GLabel 3750 3650 0    50   Input ~ 0
+$Comp
+L SparkFun-Connectors:CONN_04 J3
+U 1 1 61EE25CD
+P 4850 3550
+F 0 "J3" H 4808 4160 45  0000 C CNN
+F 1 "CONN_04" H 4808 4076 45  0000 C CNN
+F 2 "Connector_PinHeader_2.54mm:PinHeader_1x04_P2.54mm_Vertical" H 4850 4050 20  0001 C CNN
+F 3 "" H 4850 3550 50  0001 C CNN
+F 4 "CONN-09696" H 4808 3981 60  0000 C CNN "Field4"
+	1    4850 3550
+	1    0    0    -1
+$EndComp
+Text GLabel 4000 3250 2    50   Input ~ 0
+3V3
+Text GLabel 5200 3250 2    50   Input ~ 0
+3V3
+Text GLabel 4000 3350 2    50   Input ~ 0
 SDA
-Wire Wire Line
-	4050 3750 3900 3750
-Wire Wire Line
-	3900 3750 3900 3650
-Connection ~ 3900 3650
-Wire Wire Line
-	3900 3650 3750 3650
-Text GLabel 4850 3750 2    50   Input ~ 0
+Text GLabel 5200 3350 2    50   Input ~ 0
+SDA
+Text GLabel 4000 3450 2    50   Input ~ 0
 SCL
-Text GLabel 4850 3550 2    50   Input ~ 0
+Text GLabel 5200 3450 2    50   Input ~ 0
+SCL
+Text GLabel 4000 3550 2    50   Input ~ 0
 GND
-Wire Wire Line
-	4550 3750 4700 3750
-Wire Wire Line
-	4550 3650 4700 3650
-Wire Wire Line
-	4700 3650 4700 3750
-Connection ~ 4700 3750
-Wire Wire Line
-	4550 3550 4700 3550
-Wire Wire Line
-	4550 3450 4700 3450
-Wire Wire Line
-	4700 3450 4700 3550
-Connection ~ 4700 3550
-Wire Wire Line
-	4700 3550 4850 3550
-Wire Wire Line
-	4700 3750 4850 3750
+Text GLabel 5200 3550 2    50   Input ~ 0
+GND
+Wire Wire Line
+	3750 3250 4000 3250
+Wire Wire Line
+	3750 3350 4000 3350
+Wire Wire Line
+	3750 3450 4000 3450
+Wire Wire Line
+	3750 3550 4000 3550
+Wire Wire Line
+	4950 3250 5200 3250
+Wire Wire Line
+	4950 3350 5200 3350
+Wire Wire Line
+	4950 3450 5200 3450
+Wire Wire Line
+	4950 3550 5200 3550
 $EndSCHEMATC
